File: Hardware/NTR-MAIN-U2xx/NTR-MAIN-U2xx.kicad_pcb (KiCad board)
At the start: 2 copper layers, 33 x 40 mm, 97 parts, among them J1 Conn_01x15, J2 Conn_01x15, J3 Conn_01x05, J4 SW, Q1 2N7002K, U1 STM32F103CBT6, U2 FT24C64A, U3 TJA1051T/3, U4 YM23, U5 74AHC1G08SE-7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

Commit message: update boot and app
Parts:
- removed C11: 100nF 50V, Capacitor_SMD:C_0402_1005Metric
- removed U5: 74AHC1G08SE-7, Package_TO_SOT_SMD:SOT-353_SC-70-5
- added D8: BAT54AW, Package_TO_SOT_SMD:SOT-323_SC-70, B.Cu at (85.6, 62.2)
- added R38: 4.7KΩ, Resistor_SMD:R_0402_1005Metric, F.Cu at (83.9, 62.7)
Routing:
- net +3.3V: track 87.2 -> 85.2 mm
- net Net-(U6-TXD): track 2.12 -> 3.53 mm, vias 0 -> 1
- net /Bluetooth/BLE.RST: track 18.3 -> 16.9 mm
- net /K_LINE_Driver/TXD: track 12.2 -> 12.4 mm, vias 2 -> 1
- net /K_LINE_Driver/INT.9141: track 13.5 -> 13.4 mm, vias 2 -> 1
Other:
- board text added: "Ver 1.1rc"
- board text removed: "Ver 1.0"
