File: Hardware/NTR-MAIN-U2xx/mcu.kicad_sch (KiCad schematic)
At the start: 34 parts, among them J4 SW, Y1 16MHZ

Commit message: update boot and app
Parts:
- renumbered C21 to C26, C18 to C27, C18 to C28, C18 to C29, C18 to C30
